File: Slaves/LTC6811/12W/PCB/cell.kicad_sch (KiCad schematic)
At the start: 6 parts, among them Q2 TSM2323

Commit message: more updates
Parts:
- R47: renamed from R12; value 36 -> 28; MPN HRG3216Q-36R0-D-T1 -> HRG3216Q-28R0-D-T1
- R48: renamed from R13; MPN RC0603FR-07100RL -> RC0603JR-7W100RL
- renumbered C13 to C23, D1 to D16, Q2 to Q13, R14 to R49
